File: interface.sch (KiCad schematic (older format))
At the start: 3 parts

Commit message: Finished the interface schematic and started writing software's specification
Parts:
- removed H1: Raspberry Pi GPIO, symbol CONN_13X2
- added C1: 2200/10, ~, symbol CAPAPOL
- added C2: 2200/35, ~, symbol CAPAPOL
- added D1, D10, D11, D12, D13, D14, D15, D16, D17, D18, D19, D2, D20, D21, D22, D23, D24, D25, D26, D27, D28, D29, D3, D30, D31, D32, D33, D34, D35, D4, D5, D6, D7, D8, D9: LED, ~, symbol LED
- added EV1, EV10, EV11, EV12, EV13, EV14, EV15, EV16, EV17, EV18, EV19, EV2, EV20, EV21, EV22, EV23, EV24, EV25, EV26, EV27, EV28, EV29, EV3, EV30, EV31, EV32, EV4, EV5, EV6, EV7, EV8, EV9: SOLENOID, symbol SOLENOID
- added F1: FUSE, ~, symbol FUSE
- added K1, K2, K3: CONN_3, symbol CONN_3
- added Q1, Q2: BC547, ~, symbol NPN
- added Q3: NPN, ~, symbol NPN
- added R1: 47k, ~, symbol R
- added R10, R11, R12, R7, R8, R9: 3k3, ~, symbol R
- added R13, R2: 470R, ~, symbol R
- added R14, R6: 330R, ~, symbol R
- added R15, R16, R17, R18, R19, R20, R21, R22, R23, R24, R25, R26, R27, R28, R29, R30, R31, R32, R33, R34, R35, R36, R37, R38, R39, R40, R41, R42, R43, R44, R45, R46: 2k2, ~, symbol R
- added R3: 1k, ~, symbol R
- added R4: 10k, ~, symbol R
- added R5: R, ~, symbol R
- added RPi1: RASPBERRY_IO, symbol RASPBERRY_IO
- added S1: SHDN, ~, symbol SW
- added SW1, SW2: DIPS_03, symbol DIPS_03
- added SW3: SWITCH_DPDT, symbol SWITCH_DPDT
- added U1: Opto sensor, ~, symbol OPTO-TRANSISTOR4
- added U4, U5, U6, U7: ULN2803A, symbol ULN2803A
- added ~1: SMPS_POWER_SUPPLY, ~, symbol SMPS_POWER_SUPPLY
- gave numbers to parts that had none: 2
Connections:
- net labels added: 0005 + 0075, 3V3, Columns A-H, EV32 redundant, GPA0 - GPA7, GPB0 - GPB7, Rows 1-8, Rows 9-14,, Rows I-N + S
- net labels removed: +5V
- wire segments 3 -> 159
Other:
- moved on the sheet: U2, U3
