File: documentation/schematics/rpi2caster.sch (KiCad schematic (older format))
At the start: 30 parts

Commit message: Updated schematic...
Parts:
- added C1: 100u/40V, ~, symbol CPSMALL
- added C2: 1000u/10V, ~, symbol CPSMALL
- added L1: 100uH, ~, symbol INDUCTOR_SMALL
- added U1: LM2576, symbol LM2576
- Q2: renamed from Q?; value PNP -> BC557
- R1, R2: renamed from R?; value R -> 10k
- SW1: renamed from SW?; value SW_PUSH -> SHDN
- SW2: renamed from SW?; value SW_PUSH -> REBOOT
- gave numbers to parts that had none: 25
Connections:
- wire segments 44 -> 52
Other:
- moved on the sheet: P1

Commit message: (almost) final version of the schematic
Parts:
- removed D1, D2: LED R, ~, symbol LED
- removed D3: LED G, ~, symbol LED
- removed D4: LED R SB, ~, symbol LED
- removed D5: LED Y, ~, symbol LED
- removed Q1: OPTO_NPN, ~, symbol OPTO_NPN
- removed SW1: SHDN, ~, symbol SW_PUSH
- removed SW2: REBOOT, ~, symbol SW_PUSH
- added K1: 1WIRE, symbol CONN_3
- added P4: SERIAL, symbol CONN_4
- added P5: CONTROL, symbol CONN_7
- added P6: EMERG, symbol CONN_2
- added P7: SENSOR, symbol CONN_4
- added R13: 10k, ~, symbol R
- P2: value CONN_20X2 -> Raspberry Pi B+ GPIO
- P3: value CONN_20X2 -> 4 x Matrix BX758
- R12: value 2k2 -> 470R
- R5: value 510R -> 330R
- R6: value 330R -> 2k2
Connections:
- net labels removed: +24V, +3.3V, +5V
- wire segments 52 -> 109
Other:
- moved on the sheet: Q2, R10, R11, R3, R7, R8, R9

Commit message: Updated schematic and documentation, cleaned unneeded files
Parts:
- added C3, C4: 100n/63V, ~, symbol CSMALL
Connections:
- wire segments 109 -> 111
Changed lines of the file:
@@
 	1500 2100 650  2100
 Connection ~ 650  2100
+$Comp
+L CSMALL C3
+U 1 1 54D876D6
+P 1600 10450
+F 0 "C3" H 1625 10500 30  0000 L CNN
+F 1 "100n/63V" H 1625 10400 30  0000 L CNN
+F 2 "~" H 1600 10450 60  0000 C CNN
+F 3 "~" H 1600 10450 60  0000 C CNN
+	1    1600 10450
+	1    0    0    -1
+$EndComp
+$Comp
+L CSMALL C4
+U 1 1 54D876F3
+P 2950 7100
+F 0 "C4" H 2975 7150 30  0000 L CNN
+F 1 "100n/63V" H 2975 7050 30  0000 L CNN
+F 2 "~" H 2950 7100 60  0000 C CNN
+F 3 "~" H 2950 7100 60  0000 C CNN
+	1    2950 7100
+	1    0    0    -1
+$EndComp
+Wire Wire Line
+	1450 10350 1600 10350
+Wire Wire Line
+	1600 10550 1600 10650
+Connection ~ 1600 10650
+Connection ~ 1450 10350
+Connection ~ 2950 7200
+Connection ~ 2950 7000
 $EndSCHEMATC
